Commit message: added suport link and support_pivot joint. changed link coordinates to CAD values

File: urdf/scalebot.urdf (robot description, URDF)
Before this commit: robot scalebot, 3 links, 2 joints
Links:
- added link support; visual mesh filename=package://scalebot/meshes/support.stl scale=0.001 0.001 0.001
Joints:
- added joint support_pivot: type continuous, parent base, child support, origin xyz=-0.025 -0.15 0 rpy=0 0 0, axis 0 1 0
- joint base_to_laser_mount: origin xyz=.24 0 .18 rpy=0 0 0 -> xyz=.233 0 .183 rpy=0 0 0
- joint track_forks: origin xyz=-.4 -0.02 0 rpy=0 0 0 -> xyz=-.39 -0.0148 0 rpy=0 0 0

Commit message: fixed support system position

File: urdf/scalebot.urdf (robot description, URDF)
Before this commit: robot scalebot, 4 links, 3 joints
Joints:
- joint support_pivot: origin xyz=-0.025 -0.15 0 rpy=0 0 0 -> xyz=-0.025 0 -0.15 rpy=0 0 0
